File: hardware/logicboard/p2n-001.brd (EAGLE design)
At the start: 91 x 90 mm, 72 parts, among them IC1 74LS06N, IC2 4066N, J1 MKR, J10 1-Wire, J2 GPIO, J3 Vcc, J4** RLY2, J5 SPI, J6 LED, J7 DIN5, J8 DIN5, J9 DIN5, K1 G5V1, Q1 220mA/50V/3.5Ω, Q2 220mA/50V/3.5Ω, T1 2SC1815

Commit message: Trying to install Nano.
Parts:
- removed DISP2: MNTR, pinhead:1X04
- removed H1, H2: STAND-OFF, SparkFun-Hardware:STAND-OFF
- removed JP2: RTC, SparkFun-Connectors:1X05
- removed MC1: ARDUINOMICRO, adafruit:ARDUINOMICRO
- removed Q1, Q2: 220mA/50V/3.5Ω, SparkFun-DiscreteSemi:SOT23-3
- removed R101, R102, R103, R104: 10k, rcl:M2012
- removed RZ1***, RZ2***, VCCBRIDGE***: Inf, rcl:M2012
- removed VDDBRIDGE: 0, rcl:M2012
- added ARDUINO_NANO1: (no value), ArduinoNanoV30:ARDUINO_NANO
- added RN5: 2.2k, resistor-dil:DIL16
- IC1: value 74LS06N -> 74ALS05N
- R3: value 1k -> 3.3k
- RN1: value 10k -> 3.3k
- moved U$1 62.6 mm to (17.5, 61.5)
- moved LOGO1 29.3 mm to (9.00, 75.5), flipped to the top
Connections:
- removed net SCL3V: DISP1.8, Q1.2, R102.1, RZ1***.2
- removed net SDA3V: DISP1.7, Q2.2, R104.1, RZ2***.2
- removed net VCC/VDD: C11.1, C13.1, DISP1.5, DISP1.9, VCCBRIDGE***.1, VDDBRIDGE.1
- new net N$1: IC2.1, RN5.1
- new net N$2: IC2.4, RN5.2
- new net N$3: IC2.8, RN5.3
- new net N$4: IC2.11, RN5.4
- net ANLG0: now also ARDUINO_NANO1.4, RN5.16; no longer IC2.1, MC1.P$31
- net ANLG1: now also ARDUINO_NANO1.5, RN5.15; no longer IC2.4, MC1.P$30
- net ANLG2: now also ARDUINO_NANO1.6, RN5.14; no longer IC2.8, MC1.P$29
- net ANLG3: now also ARDUINO_NANO1.7, RN5.13; no longer IC2.11, MC1.P$28
- net AREF: now also ARDUINO_NANO1.3, R3.2, RN5.5; no longer MC1.P$32, R3.1
- net D7GATE: now also ARDUINO_NANO1.25; no longer MC1.P$6
- net DTCT0: now also ARDUINO_NANO1.20; no longer MC1.P$7
- net DTCT1: now also ARDUINO_NANO1.21; no longer MC1.P$4
- net DTCT2: now also ARDUINO_NANO1.22; no longer MC1.P$3
- net DTCT3: now also ARDUINO_NANO1.23; no longer MC1.P$1
- net GND: now also ARDUINO_NANO1.14, ARDUINO_NANO1.19, R3.1; no longer DISP2.1, JP2.2, MC1.P$12, MC1.P$21
- net GPIO0: now also ARDUINO_NANO1.26; no longer MC1.P$8
- net GPIO1: now also ARDUINO_NANO1.27; no longer MC1.P$5
- net LED0: now also ARDUINO_NANO1.1; no longer MC1.P$34
- net LED1: now also ARDUINO_NANO1.28; no longer MC1.P$2
- net MISO: now also ARDUINO_NANO1.30; no longer MC1.P$19
- net MNTR: now also ARDUINO_NANO1.10; no longer MC1.P$27
- net MOSI: now also ARDUINO_NANO1.29; no longer MC1.P$17
- net RLY: now also ARDUINO_NANO1.24; no longer MC1.P$9
- net RST: now also ARDUINO_NANO1.13, ARDUINO_NANO1.18; no longer MC1.P$13, MC1.P$22
- net RX: now also ARDUINO_NANO1.17; no longer MC1.P$14
- net SCK: no longer MC1.P$18
- net SCL: now also ARDUINO_NANO1.9, DISP1.8; no longer DISP2.3, JP2.4, MC1.P$10, Q1.3, R101.1, RZ1***.1
- net SDA: now also ARDUINO_NANO1.8, DISP1.7; no longer DISP2.4, JP2.5, MC1.P$11, Q2.3, R103.1, RZ2***.1
- net THS: now also ARDUINO_NANO1.11; no longer MC1.P$26
- net TX: now also ARDUINO_NANO1.16; no longer MC1.P$15
- net VCC: now also ARDUINO_NANO1.12; no longer C5.1, C6.1, C7.1, C8.1, C9.1, DISP2.2, IC2.14, J1.5, J10.3, J2.2, J5.2, JP2.1, MC1.P$23, OK1.8, R101.2, R103.2, RN2.1, RN3.1, SV3.13, VCCBRIDGE***.2
- net VCC/2: now also RN5.12; no longer R3.2
- net VDD: now also ARDUINO_NANO1.2, C11.1, C13.1, C5.1, C6.1, C7.1, C8.1, C9.1, DISP1.5, DISP1.9, IC2.14, J1.5, J10.3, J2.2, J5.2, OK1.8, RN2.1, RN3.1, SV3.13; no longer MC1.P$33, Q1.1, Q2.1, R102.2, R104.2, VDDBRIDGE.2
- net VIN: now also ARDUINO_NANO1.15; no longer MC1.P$20
Routing:
- net GND: track 463.7 -> 0.00 mm, vias 8 -> 0
- net VCC: track 345.0 -> 0.00 mm, vias 8 -> 0
- net V+: track 247.0 -> 0.00 mm, vias 5 -> 0
- net SCL: track 242.0 -> 0.00 mm, vias 7 -> 0
- net SDA: track 193.9 -> 0.00 mm, vias 8 -> 0
- net GPIO1: track 174.8 -> 0.00 mm
- net GPIO0: track 166.8 -> 0.00 mm, vias 4 -> 0
- net VCC/2: track 136.0 -> 0.00 mm, vias 3 -> 0
- net ANLG3: track 126.8 -> 0.00 mm, vias 7 -> 0
- net VDD: track 121.4 -> 0.00 mm, vias 6 -> 0
- net RLYOUT2: track 118.8 -> 0.00 mm, vias 1 -> 0
- net D7GATE: track 109.7 -> 0.00 mm, vias 1 -> 0
- net ANLG2: track 106.9 -> 0.00 mm, vias 7 -> 0
- net RLYOUT1: track 101.0 -> 0.00 mm, vias 3 -> 0
- net LED0A: track 100.6 -> 0.00 mm, vias 1 -> 0
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- removed copper zone on layer 1, net GND
- removed copper zone on layer 16, net GND
Other:
- board text added: "0.0.1-X"
- board text added: "74HC05"
- board text added: "Pineapple IIn"
- board text removed: "2.7.0-GM"
- board text removed: "5V"
- board text removed: "7406"
- board text removed: "Adafruit SSD1306"
- board text removed: "Arduino Micro"
- board text removed: "DISP"
- board text removed: "Pineapple IIb"
- board text removed: "RTC"
- board text removed: "SparkFun Real Time Clock Module (12708)"

Commit message: First try.
Connections:
- net VCC: no longer RN4.3, RN4.5, RN4.7
- net VDD: now also RN4.3, RN4.5, RN4.7
Routing:
- net GND: track 0.00 -> 450.4 mm, vias 0 -> 3
- net VDD: track 0.00 -> 333.8 mm, vias 0 -> 6
- net VCC/2: track 0.00 -> 187.5 mm, vias 0 -> 5
- net V+: track 0.00 -> 186.2 mm, vias 0 -> 7
- net SCL: track 0.00 -> 181.9 mm, vias 0 -> 6
- net SDA: track 0.00 -> 169.2 mm, vias 0 -> 9
- net VCC: track 0.00 -> 164.5 mm, vias 0 -> 4
- net N$3: track 0.00 -> 158.8 mm
- net GPIO0: track 0.00 -> 149.2 mm, vias 0 -> 4
- net GPIO1: track 0.00 -> 148.0 mm, vias 0 -> 5
- net LED0: track 0.00 -> 134.5 mm
- net LED1A: track 0.00 -> 118.8 mm, vias 0 -> 1
- net D7GATE: track 0.00 -> 117.7 mm, vias 0 -> 3
- net THS: track 0.00 -> 105.9 mm, vias 0 -> 3
- net N$2: track 0.00 -> 105.8 mm, vias 0 -> 5
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