File: hardware/logicboard/p2n-001.brd (EAGLE design)
At the start: 91 x 90 mm, 59 parts, among them IC1 74ALS05N, IC2 4066N, J1 MKR, J10 1-Wire, J2 GPIO, J3 Vcc, J4** RLY2, J5 SPI, J6 LED, J7 DIN5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

Commit message: Silk.
Parts:
- moved U$1 0.50 mm to (17.5, 61.0)
Changed lines of the file:
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@@
 <circle x="14.5" y="14" radius="2.6" width="0.2" layer="41"/>
 <circle x="76.5" y="14" radius="2.6" width="0.2" layer="41"/>
-<text x="17.5" y="60" size="1.27" layer="25" align="center">Pineapple IIn</text>
-<text x="17.5" y="58" size="1" layer="25" align="center">0.0.1-X</text>
+<text x="17.5" y="59" size="1.27" layer="25" align="center">Pineapple IIn</text>
+<text x="17.5" y="57" size="1" layer="25" align="center">0.0.1-X</text>
 <polygon width="0.15" layer="21">
 <vertex x="80.25" y="45"/>
@@
 <text x="9" y="37" size="1" layer="25" rot="R90" align="center">GPIO</text>
 <text x="37" y="88" size="1" layer="25" align="center">USB</text>
-<text x="37" y="40" size="1" layer="25" align="center">MC1</text>
+<text x="37" y="44" size="1" layer="25" align="center">MC1</text>
 <polygon width="0.1" layer="41">
 <vertex x="12" y="12.5"/>
@@
 </element>
 <element name="LOGO1" library="SparkFun-Aesthetics" package="OSHW-LOGO-S_COPPER" value="OSHW-LOGOS-COPPER" x="9" y="75.5" smashed="yes"/>
-<element name="U$1" library="pineapple" package="PINEAPPLE450_SILK" value="PINEAPPLE450_SILK" x="17.5" y="61.5" smashed="yes"/>
+<element name="U$1" library="pineapple" package="PINEAPPLE450_SILK" value="PINEAPPLE450_SILK" x="17.5" y="61" smashed="yes"/>
 <element name="K1" library="relay" library_urn="urn:adsk.eagle:library:339" package="G5V1" package3d_urn="urn:adsk.eagle:package:24341/1" value="G5V1" x="16" y="40" smashed="yes">
 <attribute name="MF" value="" x="16" y="40" size="1.778" layer="27" display="off"/>
