File: hardware/logicboard/p2n-001.sch (EAGLE design)
At the start: 72 parts, among them IC1 74LS06N, IC2 4066N, J1 MKR, J10 1-Wire, J2 GPIO, J3 Vcc, J4** RLY2, J5 SPI, J6 LED, J7 DIN5, J8 DIN5, J9 DIN5, K1 G5V1, Q1 220mA/50V/3.5Ω, Q2 220mA/50V/3.5Ω, T1 2SC1815

Commit message: Trying to install Nano.
Parts:
- removed DISP2: MNTR, pinhead:PINHD-1X4
- removed H1, H2: STAND-OFF, SparkFun-Hardware:STAND-OFF
- removed JP2: RTC, SparkFun-Connectors:CONN_05
- removed MC1: ARDUINOMICRO, adafruit:ARDUINOMICRO
- removed Q1, Q2: 220mA/50V/3.5Ω, SparkFun-DiscreteSemi:MOSFET-NCH-BSS138
- removed R101, R102, R103, R104: 10k, rcl:R-EU_M2012
- removed RZ1***, RZ2***, VCCBRIDGE***: Inf, rcl:R-EU_M2012
- removed VDDBRIDGE: 0, rcl:R-EU_M2012
- added ARDUINO_NANO1: (no value), ArduinoNanoV30:ARDUINO_NANO
- added RN5: 2.2k, resistor-dil:8R-N
- IC1: value 74LS06N -> 74ALS05N; device 74xx-us:74LS06N -> 74xx-us:74ALS05N
- R3: value 1k -> 3.3k
- RN1: value 10k -> 3.3k
Connections:
- removed net SCL3V: DISP1.8, Q1.S, R102.1, RZ1***.2
- removed net SDA3V: DISP1.7, Q2.S, R104.1, RZ2***.2
- removed net VCC/VDD: C11.1, C13.1, DISP1.5, DISP1.9, VCCBRIDGE***.1, VDDBRIDGE.1
- new net N$1: IC2A.A, RN5A.1
- new net N$2: IC2B.A, RN5B.1
- new net N$3: IC2C.A, RN5C.1
- new net N$4: IC2D.A, RN5D.1
- net ANLG0: now also ARDUINO_NANO1.A0, RN5A.2; no longer IC2A.A, MC1.A0
- net ANLG1: now also ARDUINO_NANO1.A1, RN5B.2; no longer IC2B.A, MC1.A1
- net ANLG2: now also ARDUINO_NANO1.A2, RN5C.2; no longer IC2C.A, MC1.A2
- net ANLG3: now also ARDUINO_NANO1.A3, RN5D.2; no longer IC2D.A, MC1.A3
- net AREF: now also ARDUINO_NANO1.AREF, R3.2, RN5E.1; no longer MC1.AREF, R3.1
- net D7GATE: now also ARDUINO_NANO1.D7; no longer MC1.7
- net DTCT0: now also ARDUINO_NANO1.D2; no longer MC1.6
- net DTCT1: now also ARDUINO_NANO1.D3; no longer MC1.9
- net DTCT2: now also ARDUINO_NANO1.D4; no longer MC1.10
- net DTCT3: now also ARDUINO_NANO1.D5; no longer MC1.12
- net GND: now also ARDUINO_NANO1.GND@1, ARDUINO_NANO1.GND@2, R3.1; no longer DISP2.1, JP2.2, MC1.GND, MC1.GND@1
- net GPIO0: now also ARDUINO_NANO1.D8; no longer MC1.5
- net GPIO1: now also ARDUINO_NANO1.D9; no longer MC1.8
- net LED0: now also ARDUINO_NANO1.D13; no longer MC1.13
- net LED1: now also ARDUINO_NANO1.D10; no longer MC1.11
- net MISO: now also ARDUINO_NANO1.D12; no longer MC1.MISO
- net MNTR: now also ARDUINO_NANO1.A6; no longer MC1.A4
- net MOSI: now also ARDUINO_NANO1.D11; no longer MC1.MOSI
- net RLY: now also ARDUINO_NANO1.D6; no longer MC1.4
- net RST: now also ARDUINO_NANO1.!RESET@1, ARDUINO_NANO1.!RESET@2; no longer MC1.R@1, MC1.R@2
- net RX: now also ARDUINO_NANO1.RX0; no longer MC1.RX
- net SCK: no longer MC1.SCK
- net SCL: now also ARDUINO_NANO1.A5, DISP1.8; no longer DISP2.3, JP2.4, MC1.3, Q1.D, R101.1, RZ1***.1
- net SDA: now also ARDUINO_NANO1.A4, DISP1.7; no longer DISP2.4, JP2.5, MC1.2, Q2.D, R103.1, RZ2***.1
- net THS: now also ARDUINO_NANO1.A7; no longer MC1.A5
- net TX: now also ARDUINO_NANO1.TX1; no longer MC1.TX
- net VCC: now also ARDUINO_NANO1.5V; no longer C5.1, C6.1, C7.1, C8.1, C9.1, DISP2.2, IC2P.VDD, J1.5, J10.3, J2.2, J5.2, JP2.1, MC1.5V, OK1A.VCC, R101.2, R103.2, RN2.1, RN3.1, SV3.13, VCCBRIDGE***.2
- net VCC/2: now also RN5E.2; no longer R3.2
- net VDD: now also ARDUINO_NANO1.3V3, C11.1, C13.1, C5.1, C6.1, C7.1, C8.1, C9.1, DISP1.5, DISP1.9, IC2P.VDD, J1.5, J10.3, J2.2, J5.2, OK1A.VCC, RN2.1, RN3.1, SV3.13; no longer MC1.3V, Q1.G, Q2.G, R102.2, R104.2, VDDBRIDGE.2
- net VIN: now also ARDUINO_NANO1.VIN; no longer MC1.9V
Other:
- moved on the sheet: R3

Commit message: First try.
Connections:
- net VCC: no longer RN4C.1, RN4E.1, RN4G.1
- net VDD: now also RN4C.1, RN4E.1, RN4G.1
Changed lines of the file:
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@@
 <part name="SUPPLY8" library="supply2" library_urn="urn:adsk.eagle:library:372" deviceset="VCC" device=""/>
 <part name="SUPPLY9" library="supply2" library_urn="urn:adsk.eagle:library:372" deviceset="VCC" device=""/>
-<part name="SUPPLY14" library="supply2" library_urn="urn:adsk.eagle:library:372" deviceset="VCC" device=""/>
-<part name="SUPPLY15" library="supply2" library_urn="urn:adsk.eagle:library:372" deviceset="VCC" device=""/>
 <part name="SUPPLY16" library="supply2" deviceset="GND" device=""/>
 <part name="SUPPLY17" library="supply2" deviceset="GND" device=""/>
@@
 <attribute name="VALUE" x="147.32" y="248.92" size="1.778" layer="96" align="bottom-center"/>
 </instance>
-<instance part="SUPPLY14" gate="G$1" x="170.18" y="99.06" smashed="yes">
-<attribute name="VALUE" x="170.18" y="104.14" size="1.778" layer="96" align="bottom-center"/>
-</instance>
-<instance part="SUPPLY15" gate="G$1" x="170.18" y="48.26" smashed="yes">
-<attribute name="VALUE" x="170.18" y="53.34" size="1.778" layer="96" align="bottom-center"/>
-</instance>
 <instance part="SUPPLY16" gate="GND" x="259.08" y="48.26" smashed="yes"/>
 <instance part="SUPPLY17" gate="GND" x="292.1" y="48.26" smashed="yes"/>
@@
 </segment>
 <segment>
-<pinref part="SUPPLY14" gate="G$1" pin="VCC"/>
-<wire x1="170.18" y1="96.52" x2="170.18" y2="93.98" width="0.1524" layer="91"/>
-<pinref part="RN4" gate="E" pin="1"/>
-<wire x1="172.72" y1="93.98" x2="170.18" y2="93.98" width="0.1524" layer="91"/>
-</segment>
-<segment>
-<pinref part="SUPPLY15" gate="G$1" pin="VCC"/>
-<wire x1="170.18" y1="45.72" x2="170.18" y2="43.18" width="0.1524" layer="91"/>
-<pinref part="RN4" gate="C" pin="1"/>
-<wire x1="170.18" y1="43.18" x2="170.18" y2="30.48" width="0.1524" layer="91"/>
-<wire x1="172.72" y1="43.18" x2="170.18" y2="43.18" width="0.1524" layer="91"/>
-<junction x="170.18" y="43.18"/>
-<pinref part="RN4" gate="G" pin="1"/>
-<wire x1="172.72" y1="30.48" x2="170.18" y2="30.48" width="0.1524" layer="91"/>
-</segment>
-<segment>
 <pinref part="ARDUINO_NANO1" gate="G$1" pin="5V"/>
 <wire x1="259.08" y1="152.4" x2="256.54" y2="152.4" width="0.1524" layer="91"/>
@@
 <label x="137.16" y="124.46" size="0.8128" layer="95" rot="R90" xref="yes"/>
 </segment>
-</net>
+<segment>
+<wire x1="170.18" y1="96.52" x2="170.18" y2="93.98" width="0.1524" layer="91"/>
+<pinref part="RN4" gate="E" pin="1"/>
+<wire x1="172.72" y1="93.98" x2="170.18" y2="93.98" width="0.1524" layer="91"/>
+<label x="170.18" y="96.52" size="0.8128" layer="95" rot="R90" xref="yes"/>
+</segment>
+<segment>
+<wire x1="170.18" y1="45.72" x2="170.18" y2="43.18" width="0.1524" layer="91"/>
+<pinref part="RN4" gate="C" pin="1"/>
+<wire x1="170.18" y1="43.18" x2="170.18" y2="30.48" width="0.1524" layer="91"/>
+<wire x1="172.72" y1="43.18" x2="170.18" y2="43.18" width="0.1524" layer="91"/>
+<junction x="170.18" y="43.18"/>
+<pinref part="RN4" gate="G" pin="1"/>
+<wire x1="172.72" y1="30.48" x2="170.18" y2="30.48" width="0.1524" layer="91"/>
+<label x="170.18" y="45.72" size="0.8128" layer="95" rot="R90" xref="yes"/>
+</segment>
+</net>
